File: stm32f401.kicad_pcb (KiCad board)
At the start: 2 copper layers, 35 x 35 mm, 37 parts, among them J1 USB_C_Receptacle_USB2.0_16P, SW1 SW_Push, SW2 SW_Push, U1 STM32F401RBT6, U2 BMI160, U3 AMS1117-3.3, Y1 16M

Commit message: Initial PCB Design
Parts:
- added C18: .1uF, Capacitor_SMD:C_0402_1005Metric, F.Cu at (55.1, 78.0)
- added J2: Conn_01x06_Pin, Connector_JST:JST_SH_SM06B-SRSS-TB_1x06-1MP_P1.00mm_Horizontal, F.Cu at (63.3, 53.3)
- added J3: Conn_01x04_Pin, Connector_JST:JST_SH_SM04B-SRSS-TB_1x04-1MP_P1.00mm_Horizontal, F.Cu at (50.5, 53.3)
- added SWD: Conn_01x08_Pin, Custom:Conn_0x08, F.Cu at (42.0, 80.6)
- D1: value RED -> R
- D2: value GREEN -> G
- moved H2 89.5 mm to (43.2, 53.2), turned to 90 degrees
- moved C12 88.9 mm to (45.5, 60.4)
- moved C13 88.4 mm to (45.4, 65.8)
- moved R5 86.6 mm to (34.9, 70.1), turned to 90 degrees
- moved C10 82.9 mm to (49.9, 60.1), turned to -90 degrees
- moved D2 82.4 mm to (48.5, 61.9), turned to 180 degrees
- moved C8 82.0 mm to (48.8, 67.3), turned to -90 degrees
- moved C7 80.9 mm to (49.0, 74.6)
- moved SW1 80.1 mm to (49.0, 76.9)
- moved C4 78.1 mm to (52.7, 58.0)
- moved C9 77.6 mm to (47.6, 67.3), turned to -90 degrees
- moved C11 77.5 mm to (53.1, 72.5), turned to 180 degrees
- moved SW2 75.6 mm to (49.0, 82.0)
- moved R3 75.3 mm to (48.0, 60.4), turned to -90 degrees
- moved C2 73.7 mm to (53.1, 78.0)
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Connections:
- net /NRST renamed NRST
- J1 pad S1: unconnected-(J1-SHIELD-PadS1) -> GND
- U1 pad 11: unconnected-(U1-PC3-Pad11) -> T3C4
- U1 pad 16: unconnected-(U1-PA2-Pad16) -> UART2_TX
- U1 pad 17: unconnected-(U1-PA3-Pad17) -> UART2_RX
- U1 pad 2: unconnected-(U1-PC13-Pad2) -> /USR_LED
- U1 pad 20: unconnected-(U1-PA4-Pad20) -> CS
- U1 pad 21: /USR_LED -> SCLK
- U1 pad 22: unconnected-(U1-PA6-Pad22) -> MISO
- U1 pad 23: unconnected-(U1-PA7-Pad23) -> MOSI
- U1 pad 24: unconnected-(U1-PC4-Pad24) -> T3C3
- U1 pad 25: unconnected-(U1-PC5-Pad25) -> T3C2
- U1 pad 37: unconnected-(U1-PC6-Pad37) -> T3C1
- U1 pad 46: unconnected-(U1-PA13-Pad46) -> SWDIO
- U1 pad 49: unconnected-(U1-PA14-Pad49) -> SWCLK
- U1 pad 55: unconnected-(U1-PB3-Pad55) -> SWO
- U1 pad 58: unconnected-(U1-PB6-Pad58) -> I2C1_SCL
- U1 pad 59: unconnected-(U1-PB7-Pad59) -> I2C1_SDA
Routing:
- net USB_D-: track 0.00 -> 8.65 mm
- net USB_D+: track 0.00 -> 8.65 mm
- net Net-(D1-A): track 0.00 -> 1.89 mm
Other:
- outline, holes or cut-outs redrawn
- board text added: "+"
- board text added: "-"

Commit message: Initial PCB Design
Parts:
- removed R5: 0, Resistor_SMD:R_0402_1005Metric
- added C19: .1u, Capacitor_SMD:C_0402_1005Metric, F.Cu at (67.0, 61.4)
- moved R7 2.01 mm to (67.2, 62.9)
- moved R6 0.62 mm to (66.4, 69.4)
- moved J1 0.35 mm to (72.6, 67.4)
- renumbered SWD to J5
Connections:
- C8 pad 2: /VREF -> +3V3
- C9 pad 2: /VREF -> +3V3
- U1 pad 13: /VREF -> +3V3
- U1 pad 41: unconnected-(U1-PA8-Pad41) -> INT1
- U1 pad 42: unconnected-(U1-PA9-Pad42) -> INT2
Routing:
- net USB_D-: track 8.65 -> 0.66 mm
- net USB_D+: track 8.65 -> 0.66 mm

Commit message: Initial PCB Design
Parts:
- removed C19: .1u, Capacitor_SMD:C_0402_1005Metric
- added R1: 2k2, Resistor_SMD:R_0402_1005Metric, F.Cu at (49.4, 57.2)
- added R2: 2k2, Resistor_SMD:R_0402_1005Metric, F.Cu at (51.0, 57.6)
- added U1: TPD2E2U06DCK, Package_TO_SOT_SMD:SOT-323_SC-70, F.Cu at (65.1, 66.3)
- R5: renamed from R2; value 10k -> 1k
- R6: renamed from R3; value 10k -> 1k
- moved R7 0.82 mm to (66.6, 68.6)
- moved SW2 0.39 mm to (48.9, 81.6)
- renumbered C2 to C1, C6 to C10, C7 to C11, C15 to C12, C17 to C13, C10 to C14, C11 to C15, C14 to C17, C1 to C18, C3 to C2, C9 to C3, C8 to C5, C5 to C6, C18 to C7, C12 to C8, C13 to C9, D2 to D1, D1 to D2, J3 to I2C1, J2 to PWM, R1 to R3, R6 to R7, R7 to R8, J5 to SWD, U3 to U2, U2 to U3, U1 to U4
Routing:
- net USB_D+: track 0.66 -> 11.5 mm
- net USB_D-: track 0.66 -> 9.04 mm
- net VBUS: track 0.00 -> 6.53 mm
- added copper zone on F.Cu, net VBUS

Commit message: Initial PCB Design
Parts:
- removed C11: .1uF, Capacitor_SMD:C_0402_1005Metric
- H1, H2, H3, H4: footprint MountingHole:MountingHole_2.2mm_M2_Pad_Via -> MountingHole:MountingHole_2.5mm_Pad_Via
- moved C1 3.74 mm to (53.2, 81.8)
- moved U3 3.74 mm to (54.1, 79.6)
- moved C7 3.74 mm to (55.2, 81.8)
- moved R8 2.20 mm to (67.2, 65.1)
- moved R3 1.35 mm to (50.2, 79.3)
- moved H3 1.07 mm to (72.8, 81.4)
- moved H1 0.98 mm to (72.8, 53.5)
- moved C15 0.34 mm to (52.8, 72.5)
- moved H2 0.33 mm to (43.4, 53.4)
- moved H4 0.29 mm to (43.3, 81.5)
- moved C17 0.22 mm to (62.0, 83.8)
- moved C16 0.18 mm to (62.0, 82.6)
- moved R1 0.15 mm to (49.5, 57.1)
- moved R7 0.14 mm to (66.8, 68.6)
- moved R4 0.10 mm to (54.4, 57.5)
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- renumbered SW2 to BOOT0, PWM to PWM1, SW1 to RST
Connections:
- U4 pad 26: unconnected-(U4-PB0-Pad26) -> INT1
- U4 pad 27: unconnected-(U4-PB1-Pad27) -> INT2
- U4 pad 41: INT1 -> unconnected-(U4-PA8-Pad41)
- U4 pad 42: INT2 -> unconnected-(U4-PA9-Pad42)
Routing:
- net +3V3: track 0.00 -> 150.1 mm, vias 0 -> 10
- net GND: track 0.00 -> 55.5 mm, vias 0 -> 21
- net NRST: track 0.00 -> 28.8 mm, vias 0 -> 4
- net BOOT0: track 0.00 -> 26.6 mm
- net SWCLK: track 0.00 -> 25.9 mm, vias 0 -> 2
- net SWDIO: track 0.00 -> 25.2 mm, vias 0 -> 2
- net SWO: track 0.00 -> 21.8 mm, vias 0 -> 2
- net T3C2: track 0.00 -> 18.7 mm, vias 0 -> 2
- net T3C3: track 0.00 -> 18.7 mm, vias 0 -> 2
- net T3C4: track 0.00 -> 18.0 mm, vias 0 -> 2
- net T3C1: track 0.00 -> 14.8 mm, vias 0 -> 2
- net INT1: track 0.00 -> 13.9 mm, vias 0 -> 2
- net UART2_RX: track 0.00 -> 13.2 mm, vias 0 -> 2
- net I2C1_SDA: track 0.00 -> 11.1 mm, vias 0 -> 2
- net VBUS: track 6.53 -> 17.2 mm
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- added copper zone on B.Cu, net GND
- added copper zone on F.Cu, net GND
- removed copper zone on F.Cu, net VBUS
Other:
- board size 35 x 35 mm -> 36.2 x 35 mm
