File: stm32f401.kicad_sch (KiCad schematic)
At the start: 37 parts, among them J1 USB_C_Receptacle_USB2.0_16P, SW1 SW_Push, SW2 SW_Push, U1 STM32F401RBT6, U2 BMI160, U3 AMS1117-3.3, Y1 16M

Commit message: Initial PCB Design
Parts:
- removed R5: 0, Resistor_SMD:R_0402_1005Metric, symbol Device:R_Small
- added C18: .1uF, Capacitor_SMD:C_0402_1005Metric, symbol Device:C
- added J2: Conn_01x06_Pin, Connector_JST:JST_SH_SM06B-SRSS-TB_1x06-1MP_P1.00mm_Horizontal, symbol Connector:Conn_01x06_Pin
- added J3: Conn_01x04_Pin, Connector_JST:JST_SH_SM04B-SRSS-TB_1x04-1MP_P1.00mm_Horizontal, symbol Connector:Conn_01x04_Pin
- added J5: Conn_01x08_Pin, Custom:Conn_0x08, symbol Connector:Conn_01x08_Pin
- D1: value RED -> R
- D2: value GREEN -> G
Connections:
- net VREF is gone; now on net +3V3: C8.2, C9.2, U1.13 (VREF+)
- net +3V3: now also C18.1, J2.6 (Pin_6), J3.4 (Pin_4), J5.1 (Pin_1)
- net CS: now also U1.20 (PA4)
- net GND: now also J1.S1 (SHIELD), C18.2, J2.1 (Pin_1), J3.1 (Pin_1), J5.4 (Pin_4)
- net INT1: now also U1.41 (PA8)
- net INT2: now also U1.42 (PA9)
- net MISO: now also U1.22 (PA6)
- net MOSI: now also U1.23 (PA7)
- net NRST: now also J5.5 (Pin_5)
- net SCLK: now also U1.21 (PA5)
- net USR_LED: now also U1.2 (PC13); no longer U1.21 (PA5)
- net T3C4: now reaches U1.11 (PC3)
- net T3C4: now also J2.5 (Pin_5)
- net UART2_TX: now reaches U1.16 (PA2)
- net UART2_TX: now also J5.7 (Pin_7)
- net UART2_RX: now reaches U1.17 (PA3)
- net UART2_RX: now also J5.8 (Pin_8)
- net T3C3: now reaches U1.24 (PC4)
- net T3C3: now also J2.4 (Pin_4)
- net T3C2: now reaches U1.25 (PC5)
- net T3C2: now also J2.3 (Pin_3)
- net T3C1: now reaches U1.37 (PC6)
- net T3C1: now also J2.2 (Pin_2)
- net SWDIO: now reaches U1.46 (PA13)
- net SWDIO: now also J5.2 (Pin_2)
- net SWCLK: now reaches U1.49 (PA14)
- net SWCLK: now also J5.3 (Pin_3)
- net SWO: now reaches U1.55 (PB3)
- net SWO: now also J5.6 (Pin_6)
- net I2C1_SCL: now reaches U1.58 (PB6)
- net I2C1_SCL: now also J3.2 (Pin_2)
- net I2C1_SDA: now reaches U1.59 (PB7)
- net I2C1_SDA: now also J3.3 (Pin_3)
- no-connect marks 6 -> 34
Other:
- note added: "BMI160-IMU"
- note added: "BOOT0 SW"
- note added: "Crystal"
- note added: "I2C1 Connector"
- note added: "LDO Circuit"
- note added: "Mounting Hole"
- note added: "POWER STATUS LED"
- note added: "PWM Outputs"
- note added: "RESET SW"
- note added: "SWD + UART Connector"
- note added: "USB Type-C Connector"
- note added: "USER LED"
- note added: "VDD Decoupling"
- note added: "VREF Decoupling"
- moved on the sheet: C1, C10, C11, C12, C13, C14, C15, C16, C17, C5, C6, C7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

Commit message: Initial PCB Design
Parts:
- added R1, R2: 2k2, Resistor_SMD:R_0402_1005Metric, symbol Device:R
- added U1: TPD2E2U06DCK, Package_TO_SOT_SMD:SOT-323_SC-70, symbol Power_Protection:TPD2E2U06DCK
- R5: renamed from R2; value 10k -> 1k
- R6: renamed from R3; value 10k -> 1k
- renumbered C2 to C1, C6 to C10, C7 to C11, C15 to C12, C17 to C13, C10 to C14, C11 to C15, C14 to C17, C1 to C18, C3 to C2, C9 to C3, C8 to C5, C5 to C6, C18 to C7, C12 to C8, C13 to C9, D2 to D1, D1 to D2, J3 to I2C1, J2 to PWM1, R1 to R3, R6 to R7, R7 to R8, J5 to SWD1, U3 to U2, U2 to U3, U1 to U4
Connections:
- net +3V3: now also R1.2, R2.2
- net GND: now also U1.3
- net I2C1_SCL: now also R2.1
- net I2C1_SDA: now also R1.1
- net USB_D+: now also U1.1
- net USB_D-: now also U1.2
Other:
- note added: "I2C PullUP"
- note added: "USB ESD Protection"

Commit message: Initial PCB Design
Parts:
- removed C11: .1uF, Capacitor_SMD:C_0402_1005Metric, symbol Device:C
- H1, H2, H3, H4: footprint MountingHole:MountingHole_2.2mm_M2_Pad_Via -> MountingHole:MountingHole_2.5mm_Pad_Via
Connections:
- net INT1: now also U4.26 (PB0); no longer U4.41 (PA8)
- net INT2: now also U4.27 (PB1); no longer U4.42 (PA9)
Other:
- title: (none) -> STM32F401_FC
Changed lines of the file:
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@@
 	(generator_version "9.0")
 	(paper "A4")
+	(title_block
+		(title "STM32F401_FC")
+		(rev "1.0")
+	)
 	(text "Mounting Hole\n"
 		(exclude_from_sim no)
@@
 	)
 	(junction
-		(at 97.79 175.26)
-		(diameter 0)
-		(color 0 0 0 0)
-	)
-	(junction
 		(at 173.99 93.98)
 		(diameter 0)
@@
 	)
 	(no_connect
+		(at 256.54 69.85)
+	)
+	(no_connect
 		(at 179.07 132.08)
 	)
@@
 	)
 	(no_connect
-		(at 256.54 95.25)
-	)
-	(no_connect
 		(at 256.54 74.93)
 	)
 	(no_connect
-		(at 256.54 92.71)
+		(at 256.54 72.39)
 	)
 	(no_connect
@@
 	(wire
 		(pts
-			(xy 256.54 69.85) (xy 262.89 69.85)
-		)
-		(stroke
-			(width 0)
-			(type default)
-		)
-	)
-	(wire
-		(pts
 			(xy 109.22 175.26) (xy 110.49 175.26)
 		)
@@
 	(wire
 		(pts
-			(xy 97.79 180.34) (xy 97.79 175.26)
-		)
-		(stroke
-			(width 0)
-			(type default)
-		)
-	)
-	(wire
-		(pts
 			(xy 191.77 27.94) (xy 191.77 29.21)
 		)
@@
 	(wire
 		(pts
-			(xy 100.33 180.34) (xy 97.79 180.34)
-		)
-		(stroke
-			(width 0)
-			(type default)
-		)
-	)
-	(wire
-		(pts
 			(xy 172.72 85.09) (xy 173.99 85.09)
 		)
@@
 	(wire
 		(pts
-			(xy 96.52 175.26) (xy 97.79 175.26)
+			(xy 96.52 175.26) (xy 99.06 175.26)
 		)
 		(stroke
@@
 	(wire
 		(pts
-			(xy 256.54 72.39) (xy 262.89 72.39)
-		)
-		(stroke
-			(width 0)
-			(type default)
-		)
-	)
-	(wire
-		(pts
 			(xy 41.91 22.86) (xy 52.07 22.86)
 		)
@@
 	(wire
 		(pts
-			(xy 97.79 175.26) (xy 99.06 175.26)
-		)
-		(stroke
-			(width 0)
-			(type default)
-		)
-	)
-	(wire
-		(pts
 			(xy 213.36 110.49) (xy 220.98 110.49)
 		)
@@
 	(wire
 		(pts
+			(xy 256.54 92.71) (xy 259.08 92.71)
+		)
+		(stroke
+			(width 0)
+			(type default)
+		)
+	)
+	(wire
+		(pts
 			(xy 167.64 116.84) (xy 168.91 116.84)
 		)
@@
 	(wire
 		(pts
-			(xy 107.95 180.34) (xy 110.49 180.34)
-		)
-		(stroke
-			(width 0)
-			(type default)
-		)
-	)
-	(wire
-		(pts
 			(xy 165.1 92.71) (xy 165.1 93.98)
 		)
@@
 	(wire
 		(pts
+			(xy 256.54 95.25) (xy 259.08 95.25)
+		)
+		(stroke
+			(width 0)
+			(type default)
+		)
+	)
+	(wire
+		(pts
 			(xy 67.31 49.53) (xy 67.31 50.8)
 		)
@@
 	(wire
 		(pts
-			(xy 110.49 180.34) (xy 110.49 175.26)
-		)
-		(stroke
-			(width 0)
-			(type default)
-		)
-	)
-	(wire
-		(pts
 			(xy 67.31 43.18) (xy 73.66 43.18)
 		)
@@
 		)
 	)
-	(global_label "INT2"
-		(shape input)
-		(at 262.89 72.39 0)
-		(fields_autoplaced yes)
-		(effects
-			(font
-				(size 1.27 1.27)
-			)
-			(justify left)
-		)
-		(property "Intersheetrefs" "${INTERSHEET_REFS}"
-			(at 269.9876 72.39 0)
-			(effects
-				(font
-					(size 1.27 1.27)
-				)
-				(justify left)
-				(hide yes)
-			)
-		)
-	)
 	(global_label "INT1"
 		(shape input)
@@
 		)
 	)
+	(global_label "INT2"
+		(shape input)
+		(at 259.08 95.25 0)
+		(fields_autoplaced yes)
+		(effects
+			(font
+				(size 1.27 1.27)
+			)
+			(justify left)
+		)
+		(property "Intersheetrefs" "${INTERSHEET_REFS}"
+			(at 266.1776 95.25 0)
+			(effects
+				(font
+					(size 1.27 1.27)
+				)
+				(justify left)
+				(hide yes)
+			)
+		)
+	)
 	(global_label "CS"
 		(shape input)
@@
 		)
 	)
-	(global_label "INT1"
-		(shape input)
-		(at 262.89 69.85 0)
-		(fields_autoplaced yes)
-		(effects
-			(font
-				(size 1.27 1.27)
-			)
-			(justify left)
-		)
-		(property "Intersheetrefs" "${INTERSHEET_REFS}"
-			(at 269.9876 69.85 0)
-			(effects
-				(font
-					(size 1.27 1.27)
-				)
-				(justify left)
-				(hide yes)
-			)
-		)
-	)
 	(global_label "NRST"
 		(shape input)
@@
 		)
 	)
+	(global_label "INT1"
+		(shape input)
+		(at 259.08 92.71 0)
+		(fields_autoplaced yes)
+		(effects
+			(font
+				(size 1.27 1.27)
+			)
+			(justify left)
+		)
+		(property "Intersheetrefs" "${INTERSHEET_REFS}"
+			(at 266.1776 92.71 0)
+			(effects
+				(font
+					(size 1.27 1.27)
+				)
+				(justify left)
+				(hide yes)
+			)
+		)
+	)
 	(global_label "INT2"
 		(shape input)
@@
 			)
 		)
-		(property "Footprint" "MountingHole:MountingHole_2.2mm_M2_Pad_Via"
+		(property "Footprint" "MountingHole:MountingHole_2.5mm_Pad_Via"
 			(at 21.59 175.26 0)
 			(effects
@@
 	)
 	(symbol
-		(lib_id "Device:C")
-		(at 104.14 180.34 90)
-		(mirror x)
-		(unit 1)
-		(exclude_from_sim no)
-		(in_bom yes)
-		(on_board yes)
-		(dnp no)
-		(property "Reference" "C11"
-			(at 104.14 187.96 90)
-			(effects
-				(font
-					(size 1.27 1.27)
-				)
-			)
-		)
-		(property "Value" ".1uF"
-			(at 104.14 185.42 90)
-			(effects
-				(font
-					(size 1.27 1.27)
-				)
-			)
-		)
-		(property "Footprint" "Capacitor_SMD:C_0402_1005Metric"
-			(at 107.95 181.3052 0)
-			(effects
-				(font
-					(size 1.27 1.27)
-				)
-				(hide yes)
-			)
-		)
-		(property "Datasheet" "~"
-			(at 104.14 180.34 0)
-			(effects
-				(font
-					(size 1.27 1.27)
-				)
-				(hide yes)
-			)
-		)
-		(property "Description" "Unpolarized capacitor"
-			(at 104.14 180.34 0)
-			(effects
-				(font
-					(size 1.27 1.27)
-				)
-				(hide yes)
-			)
-		)
-		(pin "1"
-		)
-		(pin "2"
-		)
-		(instances
-			(project "stm32f401"
-				(path "/b3a87104-3d12-4882-9351-41db6a7a6647"
-					(reference "C11")
-					(unit 1)
-				)
-			)
-		)
-	)
-	(symbol
 		(lib_id "Sensor_Motion:BMI160")
 		(at 168.91 129.54 0)
@@
 			)
 		)
-		(property "Footprint" "MountingHole:MountingHole_2.2mm_M2_Pad_Via"
+		(property "Footprint" "MountingHole:MountingHole_2.5mm_Pad_Via"
 			(at 21.59 162.56 0)
 			(effects
@@
 			)
 		)
-		(property "Footprint" "MountingHole:MountingHole_2.2mm_M2_Pad_Via"
+		(property "Footprint" "MountingHole:MountingHole_2.5mm_Pad_Via"
 			(at 21.59 181.61 0)
 			(effects
@@
 			)
 		)
-		(property "Footprint" "MountingHole:MountingHole_2.2mm_M2_Pad_Via"
+		(property "Footprint" "MountingHole:MountingHole_2.5mm_Pad_Via"
 			(at 21.59 168.91 0)
 			(effects
